File: M2S-v2-Modular.brd (EAGLE design)
At the start: 55 x 40 mm, 75 parts, among them J5 Qwiic Right Angle, J6 SM05B-SRSS-TB, U1 INA333AIDGKT, U2 LMV324, U3 INA333AIDGKT, U4 INA333AIDGKT, U5 INA333AIDGKT, U6 REF2033AIDDCT, U7 ADS1115IDGST

Commit message: ADC Fix
Changed ADC from ADS1115 to ADS1015.

Added EAGLE libraries.

Updated/Fixed JLCPCB BOM and PnP files.

Added PDF for the schematics for easier access.
Parts:
- U7: value ADS1115IDGST -> ADS1015IDGST; device ADS1115IDGST:SOP50P490X110-10N -> ADS1015IDGST:SOP50P490X110-10N

Commit message: Fix ESLOV Pinout
Fixed ESLOV Pinout, swapped SDA and INT pins.
Connections:
- net RDY: now also J6.2; no longer J6.4
- net SDA: now also J6.4; no longer J6.2
Routing:
- net SDA: track 35.6 -> 41.7 mm, vias 2 -> 4
- net RDY: track 32.6 -> 28.6 mm
Changed lines of the file:
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@@
 <wire x1="41.5" y1="21.5" x2="44" y2="24" width="0.28" layer="1"/>
 <contactref element="R29" pad="1"/>
-<contactref element="J6" pad="2"/>
-<wire x1="43" y1="10.92" x2="43" y2="10" width="0.44" layer="1"/>
-<wire x1="43" y1="10" x2="44" y2="9" width="0.44" layer="1"/>
-<wire x1="44" y1="9" x2="44" y2="6.175" width="0.44" layer="1"/>
-<wire x1="41.5" y1="18" x2="44.25" y2="15.25" width="0.28" layer="1"/>
-<wire x1="43.67" y1="10.92" x2="43" y2="10.92" width="0.28" layer="1"/>
-<wire x1="44.25" y1="15.25" x2="44.25" y2="11.5" width="0.28" layer="1"/>
-<wire x1="44.25" y1="11.5" x2="43.67" y2="10.92" width="0.28" layer="1"/>
 <contactref element="U7" pad="9"/>
-<wire x1="41.5" y1="19.85" x2="41.5" y2="18" width="0.28" layer="1"/>
 <wire x1="41.5" y1="19.85" x2="41.5" y2="21.5" width="0.28" layer="1"/>
+<contactref element="J6" pad="4"/>
+<wire x1="43" y1="10.92" x2="43" y2="9.5" width="0.44" layer="1"/>
+<via x="43" y="9.5" extent="1-16" drill="0.35"/>
+<wire x1="43" y1="9.5" x2="46" y2="9.5" width="0.44" layer="16"/>
+<via x="46" y="9.5" extent="1-16" drill="0.35"/>
+<wire x1="46" y1="9.5" x2="46" y2="24" width="0.44" layer="1"/>
+<wire x1="46" y1="6.175" x2="46" y2="9.5" width="0.44" layer="1"/>
 </signal>
 <signal name="RDY">
 <via x="41" y="22" extent="1-16" drill="0.35"/>
 <wire x1="41.5" y1="22.5" x2="41" y2="22" width="0.28" layer="1"/>
-<wire x1="41" y1="22" x2="46" y2="22" width="0.44" layer="16"/>
-<via x="46" y="22" extent="1-16" drill="0.35"/>
+<wire x1="41" y1="22" x2="44" y2="22" width="0.44" layer="16"/>
+<via x="44" y="22" extent="1-16" drill="0.35"/>
 <contactref element="R31" pad="1"/>
-<via x="46" y="7.5" extent="1-16" drill="0.35"/>
-<wire x1="46" y1="7.5" x2="40" y2="7.5" width="0.44" layer="16"/>
+<via x="44" y="7.5" extent="1-16" drill="0.35"/>
+<wire x1="44" y1="7.5" x2="40" y2="7.5" width="0.44" layer="16"/>
 <via x="40" y="7.5" extent="1-16" drill="0.35"/>
 <wire x1="40" y1="7.5" x2="40" y2="10.92" width="0.44" layer="1"/>
-<contactref element="J6" pad="4"/>
-<wire x1="46" y1="7.5" x2="46" y2="6.175" width="0.44" layer="1"/>
-<wire x1="46" y1="22" x2="46" y2="7.5" width="0.44" layer="1"/>
+<wire x1="44" y1="22" x2="44" y2="7.5" width="0.44" layer="1"/>
 <contactref element="U7" pad="2"/>
 <wire x1="41.5" y1="24.15" x2="41.5" y2="22.5" width="0.28" layer="1"/>
+<contactref element="J6" pad="2"/>
+<wire x1="44" y1="6.175" x2="44" y2="7.5" width="0.44" layer="1"/>
 </signal>
 </signals>
